File: KiCAD/plate kicad files/vault35-katana plate_universal.kicad_pcb (KiCad board)
At the start: 2 copper layers, 210.6 x 77.3 mm, 0 parts

Commit message: update plates
Other:
- outline, holes or cut-outs redrawn
Changed lines of the file:
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@@
   (gr_curve (pts (xy 185.457844 104.368479) (xy 185.457844 104.086363) (xy 185.210989 103.839513) (xy 184.928878 103.839513))
     (stroke (width 0.2) (type solid)) (layer "Edge.Cuts"))
-  (gr_curve (pts (xy 250.873317 58.771605) (xy 250.873317 58.48949) (xy 250.661718 58.277905) (xy 250.379607 58.277905))
-    (stroke (width 0.2) (type solid)) (layer "Edge.Cuts"))
   (gr_line (start 196.38981 81.235032) (end 196.38981 68.25773)
     (stroke (width 0.2) (type solid)) (layer "Edge.Cuts"))
-  (gr_line (start 250.379607 58.277905) (end 248.47532 58.277905)
-    (stroke (width 0.2) (type solid)) (layer "Edge.Cuts"))
   (gr_line (start 215.432589 81.235032) (end 215.432589 68.25773)
     (stroke (width 0.2) (type solid)) (layer "Edge.Cuts"))
@@
   (gr_curve (pts (xy 67.851046 100.313078) (xy 67.851046 100.595194) (xy 68.062632 100.806777) (xy 68.344748 100.806777))
     (stroke (width 0.2) (type solid)) (layer "Edge.Cuts"))
-  (gr_curve (pts (xy 248.47532 49.214952) (xy 248.47532 48.932836) (xy 248.193209 48.72125) (xy 247.805288 48.72125))
+  (gr_curve (pts (xy 250.855 49.208297) (xy 250.855 48.926181) (xy 250.572889 48.714595) (xy 250.184968 48.714595))
     (stroke (width 0.2) (type solid)) (layer "Edge.Cuts"))
   (gr_curve (pts (xy 86.893825 100.313078) (xy 86.893825 100.595194) (xy 87.105411 100.806777) (xy 87.387527 100.806777))
@@
   (gr_line (start 49.689878 100.806777) (end 62.314535 100.806777)
     (stroke (width 0.2) (type solid)) (layer "Edge.Cuts"))
-  (gr_line (start 248.47532 58.277905) (end 248.47532 49.214952)
+  (gr_line (start 250.855 58.27125) (end 250.855 49.208297)
     (stroke (width 0.2) (type solid)) (layer "Edge.Cuts"))
   (gr_curve (pts (xy 105.160788 67.764028) (xy 105.442904 67.764028) (xy 105.654488 67.975613) (xy 105.654488 68.25773))
@@
   (gr_curve (pts (xy 138.485652 100.806777) (xy 138.767763 100.806777) (xy 138.979351 100.595189) (xy 138.979351 100.313078))
     (stroke (width 0.2) (type solid)) (layer "Edge.Cuts"))
-  (gr_line (start 247.805288 48.72125) (end 237.895998 48.72125)
+  (gr_line (start 250.184968 48.714595) (end 237.895998 48.72125)
     (stroke (width 0.2) (type solid)) (layer "Edge.Cuts"))
   (gr_curve (pts (xy 115.457999 49.214952) (xy 115.457999 48.932836) (xy 115.669588 48.72125) (xy 115.951698 48.72125))
@@
   (gr_curve (pts (xy 71.694867 62.685955) (xy 72.082774 62.685955) (xy 72.364891 62.474369) (xy 72.364891 62.192253))
     (stroke (width 0.2) (type solid)) (layer "Edge.Cuts"))
-  (gr_line (start 250.873317 71.748906) (end 250.873317 58.771605)
+  (gr_line (start 250.873317 71.748906) (end 250.855 58.27125)
     (stroke (width 0.2) (type solid)) (layer "Edge.Cuts"))
   (gr_curve (pts (xy 202.66687 105.814322) (xy 202.384759 105.814322) (xy 202.137904 105.567472) (xy 202.137904 105.285356))
@@
       24362a4a-a1be-4931-b60a-68fa25cc2703
       259695e8-0690-42a2-a863-d2fb7aeb28a1
-      25f3eec0-08d7-49a1-8cb4-424f99759664
       26758b45-428d-4d42-a099-24f154112753
-      268d0a93-80fb-4a0a-9b62-2cb3fbac4430
       2962e974-10d2-4eae-8fbe-00a1e17aa0c0
       29f02be2-a17a-41e7-9094-ac46100e77fd
