File: KiCAD/vault35-katana-sk6812/vault35-katana-sk6812.kicad_sch (KiCad schematic)
At the start: 137 parts, among them J1 USB_C_Receptacle_USB2.0, SW36 Rotary_Encoder_Switch, U1 STM32F072CBT6, U2 PRTR5V0U2X

Commit message: update plates
Parts:
- C? (x9): Package (none) -> C_0402
- C?: Package (none) -> C_0603
- D1, D10, D11, D12, D13, D14, D15, D16, D17, D18, D19, D2, D20, D21, D22, D23, D24, D25, D26, D27, D28, D29, D3, D30, D31, D32, D33, D34, D35, D36, D37, D38, D39, D4, D5, D6, D7, D8, D9: Package (none) -> SOD-123
- D107, D108, D109, D110, D111, J1, SW?: Package (none) -> SMD
- F1: Package (none) -> F_1206
- L1: Package L1206 -> L_1206
- R? (x4): Package (none) -> R_0402
- U1: Package (none) -> LQFP-48(7x7)
- U2: Package (none) -> SOD-143
- U?: Package (none) -> SOT-23-3L
